File: KiCad/AA-W6EEN.kicad_sch (KiCad schematic)
At the start: 68 parts, among them J1 ANT, J2 BATT-MODULE, J3 2.4" TFT with EC11, Q1 BF998, Q2 AO3401A, Q3 MMBT2222A, T1 Bifilar-10T, U1 Si5351A-B-GT, U2 LM358, U3 AMS1117-3.3

Commit message: Updated OPAMP footprint. Changed date/revision.
Parts:
- U2: footprint Package_SO:SOIC-8_5.3x5.3mm_P1.27mm -> MY-SOIC8:My-SOIC8
Changed lines of the file:
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@@
 	(text "STEP-IN"
 		(exclude_from_sim no)
-		(at 150.368 119.888 0)
+		(at 150.622 116.84 0)
 		(effects
 			(font
@@
 	(text "CHG-OUT"
 		(exclude_from_sim no)
-		(at 150.368 116.84 0)
+		(at 150.114 119.634 0)
 		(effects
 			(font
@@
 			)
 		)
-		(property "Footprint" "Package_SO:SOIC-8_5.3x5.3mm_P1.27mm"
+		(property "Footprint" "MY-SOIC8:My-SOIC8"
 			(at 127 57.15 0)
 			(effects
@@
 			)
 		)
-		(property "Footprint" "Package_SO:SOIC-8_5.3x5.3mm_P1.27mm"
+		(property "Footprint" "MY-SOIC8:My-SOIC8"
 			(at 106.68 54.61 0)
 			(effects
@@
 			)
 		)
-		(property "Footprint" "Package_SO:SOIC-8_5.3x5.3mm_P1.27mm"
+		(property "Footprint" "MY-SOIC8:My-SOIC8"
 			(at 127 57.15 0)
 			(effects
